Commit message: paralelepipedo

File: robotao_description/urdf/robotao.urdf.xacro (robot description, xacro)
@@ -170,5 +170,5 @@
         <inertial>
             <origin xyz="0 0 0" rpy="0 0 0"/>
-            <mass value="5.5"/>
+            <mass value="15"/>
             <inertia ixx="1.0" ixy="0.0" ixz="0.0" iyy="1.0" iyz="0.0" izz="1.0" />
         </inertial>
@@ -259,5 +259,5 @@
 <link name="torso_link">
     <visual>
-        <origin xyz="0 0 ${-0.02}" rpy="0 0 0"/>
+        <origin xyz="0 0 -0.02" rpy="0 0 0"/>
         <geometry>
             <!--<cylinder radius="${torso_radius}" length="${torso_height}" />-->
@@ -277,4 +277,65 @@
     </inertial>
 </link>
+<link name="hokuyo_link">
+    <visual>
+        <origin xyz="0 0 0" rpy="0 0 0"/>
+        <geometry>
+            <mesh filename="package://robotao_description/meshes/hokuyo.dae"/>
+        </geometry>
+    </visual>
+    <collision>
+        <origin xyz="0 0 0" rpy="0 0 0"/>
+        <geometry>
+            <mesh filename="package://robotao_description/meshes/hokuyo.dae"/>
+        </geometry>
+    </collision>
+    <inertial>
+        <origin xyz="0 0 0" rpy="0 0 0"/>
+        <mass value="1.0"/>
+        <inertia ixx="1.0" ixy="0.0" ixz="0.0" iyy="1.0" iyz="0.0" izz="1.0" />
+    </inertial>
+</link>
+<joint name="hokuyo_joint" type="fixed">
+    <axis xyz="0 0 0"/>
+    <parent link="torso_link"/>
+    <child  link="hokuyo_link"/>
+    <origin xyz="0  0 ${+torso_height/2}" rpy="0 0 0" />
+</joint>
+<!-- hokuyo -->
+<gazebo reference="hokuyo_link">
+<sensor type="gpu_ray" name="head_hokuyo_sensor">
+    <pose>0 0 0 0 0 0</pose>
+    <visualize>true</visualize>
+    <update_rate>40</update_rate>
+    <ray>
+    <scan>
+        <horizontal>
+        <samples>360</samples>
+        <resolution>1</resolution>
+        <min_angle>-3.141592654</min_angle>
+        <max_angle>3.141592654</max_angle>
+        </horizontal>
+    </scan>
+    <range>
+        <min>0.10</min>
+        <max>3.0</max>
+        <resolution>0.01</resolution>
+    </range>
+    <noise>
+        <type>gaussian</type>
+        <!-- Noise parameters based on published spec for Hokuyo laser
+            achieving "+-30mm" accuracy at range < 10m.  A mean of 0.0m and
+            stddev of 0.01m will put 99.7% of samples within 0.03m of the true
+            reading. -->
+        <mean>0.0</mean>
+        <stddev>0.01</stddev>
+    </noise>
+    </ray>
+    <plugin name="gazebo_ros_head_hokuyo_controller" filename="libgazebo_ros_gpu_laser.so">
+    <topicName>/robotao/laser/scan</topicName>
+    <frameName>hokuyo_link</frameName>
+    </plugin>
+</sensor>
+</gazebo>
 <!-- Freeze the robot in place -->
 <gazebo>
